Commit message: Fix barret urdf to comply with mujoco xml used to generate poses, change orientation order from rxyz to sxyz

File: source/IsaacGraspEnv/IsaacGraspEnv/robots/hand_barret/bh_alone.urdf (robot description, URDF)
Before this commit: robot bhand, 17 links, 16 joints
Joints:
- joint base_joint_R: child root_link_4 -> base_link; limit lower=0 upper=6.28 effort=1000 velocity=2 -> lower=-6.28 upper=6.28 effort=1000 velocity=2; parent root_link_3 -> root_link_5
- joint base_joint_Y: child base_link -> root_link_4; parent root_link_5 -> root_link_3
- joint bh_base_joint: origin xyz=0 0 0 rpy=0 0 0 -> xyz=0 0 -0.12 rpy=0 0 0
